Commit message: [Minor] 関節の配置（方向）を変更。(develop)

File: robots/robot.urdf.xacro (robot description, xacro)
@@ -4,4 +4,5 @@
   <xacro:include filename="$(find lily_octpus_description)/urdf/leg/leg.urdf.xacro"/>
   <xacro:include filename="$(find lily_octpus_description)/urdf/params/robot.xacro"/>
+  <!--
   <link name="world"/>
   <joint name="fixed" type="fixed">
@@ -9,4 +10,5 @@
     <child link="base_footprint"/>
   </joint>
+  -->
   <!-- ===============  Link & Joint =============== -->
   <!-- Base -->
@@ -21,40 +23,40 @@
   </xacro:base>
   <!-- LEG -->
-  <xacro:leg prefix="BLF" parent="base_link" origin_xyz="${body_length/2} ${body_width/2} ${-body_height/2}" origin_rpy="0.955316618 0.0 ${-M_PI/4}"
+  <xacro:leg prefix="BLF" parent="base_link" origin_xyz="${body_length/2} ${body_width/2} ${-body_height/2}" origin_rpy="0 ${M_PI/2-0.955316618} ${M_PI/4}"
              base_clause_radius="${base_clause_radius}" base_clause_length="${LF_base_clause_length}" base_clause_rpy="${LF_base_clause_rpy}" base_clause_rho="${base_clause_rho}" base_clause_torque="${base_clause_torque}" base_clause_velocity="${base_clause_velocity}"
              thigh_radius="${thigh_radius}" thigh_length="${LF_thigh_length}" thigh_rpy="${LF_thigh_rpy}" thigh_rho="${thigh_rho}" thigh_torque="${thigh_torque}" thigh_velocity="${thigh_velocity}"
              tibia_radius="${tibia_radius}" tibia_length="${LF_tibia_length}" tibia_rpy="${LF_tibia_rpy}" tibia_rho="${tibia_rho}" tibia_torque="${tibia_torque}" tibia_velocity="${tibia_velocity}"
              appendix_radius="${appendix_radius}" appendix_rho="${appendix_rho}"/>
-	<xacro:leg prefix="BLH" parent="base_link" origin_xyz="${-body_length/2} ${body_width/2} ${-body_height/2}" origin_rpy="0.955316618 0.0 ${M_PI/4}"
+	<xacro:leg prefix="BLH" parent="base_link" origin_xyz="${-body_length/2} ${body_width/2} ${-body_height/2}" origin_rpy="0 ${M_PI/2-0.955316618} ${3*M_PI/4}"
              base_clause_radius="${base_clause_radius}" base_clause_length="${LH_base_clause_length}" base_clause_rpy="${LH_base_clause_rpy}" base_clause_rho="${base_clause_rho}" base_clause_torque="${base_clause_torque}" base_clause_velocity="${base_clause_velocity}"
              thigh_radius="${thigh_radius}" thigh_length="${LH_thigh_length}" thigh_rpy="${LH_thigh_rpy}" thigh_rho="${thigh_rho}" thigh_torque="${thigh_torque}" thigh_velocity="${thigh_velocity}"
              tibia_radius="${tibia_radius}" tibia_length="${LH_tibia_length}" tibia_rpy="${LH_tibia_rpy}" tibia_rho="${tibia_rho}" tibia_torque="${tibia_torque}" tibia_velocity="${tibia_velocity}"
              appendix_radius="${appendix_radius}" appendix_rho="${appendix_rho}"/>
-  <xacro:leg prefix="BRF" parent="base_link" origin_xyz="${body_length/2} ${-body_width/2} ${-body_height/2}" origin_rpy="0.955316618 0.0 ${-3*M_PI/4}"
+  <xacro:leg prefix="BRF" parent="base_link" origin_xyz="${body_length/2} ${-body_width/2} ${-body_height/2}" origin_rpy="0 ${M_PI/2-0.955316618} ${-M_PI/4}"
              base_clause_radius="${base_clause_radius}" base_clause_length="${RF_base_clause_length}" base_clause_rpy="${RF_base_clause_rpy}" base_clause_rho="${base_clause_rho}" base_clause_torque="${base_clause_torque}" base_clause_velocity="${base_clause_velocity}"
              thigh_radius="${thigh_radius}" thigh_length="${RF_thigh_length}" thigh_rpy="${RF_thigh_rpy}" thigh_rho="${thigh_rho}" thigh_torque="${thigh_torque}" thigh_velocity="${thigh_velocity}"
              tibia_radius="${tibia_radius}" tibia_length="${RF_tibia_length}" tibia_rpy="${RF_tibia_rpy}" tibia_rho="${tibia_rho}" tibia_torque="${tibia_torque}" tibia_velocity="${tibia_velocity}"
              appendix_radius="${appendix_radius}" appendix_rho="${appendix_rho}"/>
-	<xacro:leg prefix="BRH" parent="base_link" origin_xyz="${-body_length/2} ${-body_width/2} ${-body_height/2}" origin_rpy="0.955316618 0.0 ${3*M_PI/4}"
+	<xacro:leg prefix="BRH" parent="base_link" origin_xyz="${-body_length/2} ${-body_width/2} ${-body_height/2}" origin_rpy="0 ${M_PI/2-0.955316618} ${-3*M_PI/4}"
              base_clause_radius="${base_clause_radius}" base_clause_length="${RH_base_clause_length}" base_clause_rpy="${RH_base_clause_rpy}" base_clause_rho="${base_clause_rho}" base_clause_torque="${base_clause_torque}" base_clause_velocity="${base_clause_velocity}"
              thigh_radius="${thigh_radius}" thigh_length="${RH_thigh_length}" thigh_rpy="${RH_thigh_rpy}" thigh_rho="${thigh_rho}" thigh_torque="${thigh_torque}" thigh_velocity="${thigh_velocity}"
              tibia_radius="${tibia_radius}" tibia_length="${RH_tibia_length}" tibia_rpy="${RH_tibia_rpy}" tibia_rho="${tibia_rho}" tibia_torque="${tibia_torque}" tibia_velocity="${tibia_velocity}"
              appendix_radius="${appendix_radius}" appendix_rho="${appendix_rho}"/>
-  <xacro:leg prefix="TLF" parent="base_link" origin_xyz="${body_length/2} ${body_width/2} ${body_height/2}" origin_rpy="${M_PI+0.955316618} 0.0 ${3*M_PI/4}"
+  <xacro:leg prefix="TLF" parent="base_link" origin_xyz="${body_length/2} ${body_width/2} ${body_height/2}" origin_rpy="0 ${-M_PI/2+0.955316618} ${M_PI/4}"
              base_clause_radius="${base_clause_radius}" base_clause_length="${LF_base_clause_length}" base_clause_rpy="${LF_base_clause_rpy}" base_clause_rho="${base_clause_rho}" base_clause_torque="${base_clause_torque}" base_clause_velocity="${base_clause_velocity}"
              thigh_radius="${thigh_radius}" thigh_length="${LF_thigh_length}" thigh_rpy="${LF_thigh_rpy}" thigh_rho="${thigh_rho}" thigh_torque="${thigh_torque}" thigh_velocity="${thigh_velocity}"
              tibia_radius="${tibia_radius}" tibia_length="${LF_tibia_length}" tibia_rpy="${LF_tibia_rpy}" tibia_rho="${tibia_rho}" tibia_torque="${tibia_torque}" tibia_velocity="${tibia_velocity}"
              appendix_radius="${appendix_radius}" appendix_rho="${appendix_rho}"/>
-	<xacro:leg prefix="TLH" parent="base_link" origin_xyz="${-body_length/2} ${body_width/2} ${body_height/2}" origin_rpy="${M_PI+0.955316618} 0.0 ${-3*M_PI/4}"
+	<xacro:leg prefix="TLH" parent="base_link" origin_xyz="${-body_length/2} ${body_width/2} ${body_height/2}" origin_rpy="0 ${-M_PI/2+0.955316618} ${3*M_PI/4}"
              base_clause_radius="${base_clause_radius}" base_clause_length="${LH_base_clause_length}" base_clause_rpy="${LH_base_clause_rpy}" base_clause_rho="${base_clause_rho}" base_clause_torque="${base_clause_torque}" base_clause_velocity="${base_clause_velocity}"
              thigh_radius="${thigh_radius}" thigh_length="${LH_thigh_length}" thigh_rpy="${LH_thigh_rpy}" thigh_rho="${thigh_rho}" thigh_torque="${thigh_torque}" thigh_velocity="${thigh_velocity}"
              tibia_radius="${tibia_radius}" tibia_length="${LH_tibia_length}" tibia_rpy="${LH_tibia_rpy}" tibia_rho="${tibia_rho}" tibia_torque="${tibia_torque}" tibia_velocity="${tibia_velocity}"
              appendix_radius="${appendix_radius}" appendix_rho="${appendix_rho}"/>
-  <xacro:leg prefix="TRF" parent="base_link" origin_xyz="${body_length/2} ${-body_width/2} ${body_height/2}" origin_rpy="${M_PI+0.955316618} 0.0 ${M_PI/4}"
+  <xacro:leg prefix="TRF" parent="base_link" origin_xyz="${body_length/2} ${-body_width/2} ${body_height/2}" origin_rpy="0 ${-M_PI/2+0.955316618} ${-M_PI/4}"
              base_clause_radius="${base_clause_radius}" base_clause_length="${RF_base_clause_length}" base_clause_rpy="${RF_base_clause_rpy}" base_clause_rho="${base_clause_rho}" base_clause_torque="${base_clause_torque}" base_clause_velocity="${base_clause_velocity}"
              thigh_radius="${thigh_radius}" thigh_length="${RF_thigh_length}" thigh_rpy="${RF_thigh_rpy}" thigh_rho="${thigh_rho}" thigh_torque="${thigh_torque}" thigh_velocity="${thigh_velocity}"
              tibia_radius="${tibia_radius}" tibia_length="${RF_tibia_length}" tibia_rpy="${RF_tibia_rpy}" tibia_rho="${tibia_rho}" tibia_torque="${tibia_torque}" tibia_velocity="${tibia_velocity}"
              appendix_radius="${appendix_radius}" appendix_rho="${appendix_rho}"/>
-	<xacro:leg prefix="TRH" parent="base_link" origin_xyz="${-body_length/2} ${-body_width/2} ${body_height/2}" origin_rpy="${M_PI+0.955316618} 0.0 ${-M_PI/4}"
+	<xacro:leg prefix="TRH" parent="base_link" origin_xyz="${-body_length/2} ${-body_width/2} ${body_height/2}" origin_rpy="0 ${-M_PI/2+0.955316618} ${-3*M_PI/4}"
              base_clause_radius="${base_clause_radius}" base_clause_length="${RH_base_clause_length}" base_clause_rpy="${RH_base_clause_rpy}" base_clause_rho="${base_clause_rho}" base_clause_torque="${base_clause_torque}" base_clause_velocity="${base_clause_velocity}"
              thigh_radius="${thigh_radius}" thigh_length="${RH_thigh_length}" thigh_rpy="${RH_thigh_rpy}" thigh_rho="${thigh_rho}" thigh_torque="${thigh_torque}" thigh_velocity="${thigh_velocity}"

File: urdf/leg/leg.urdf.xacro (robot description, xacro)
@@ -23,5 +23,5 @@
                                           velocity="${base_clause_velocity}">
     <origin xyz="0.0 0.0 0.0" rpy="${base_clause_rpy}"/>
-    <axis xyz="0 0 1"/>
+    <axis xyz="1 0 0"/>
     </xacro:base_clause>
     <xacro:thigh prefix="${prefix}"
