Commit message: [Minor] パラメータ調整(develop)

File: urdf/appendix/appendix.urdf.xacro (robot description, xacro)
@@ -12,4 +12,5 @@
 	  <limit lower="-0.0" upper="0.0" effort="100" velocity="100" />
 	  <insert_block name="joint_axis"/>
+	  <dynamics friction="1.0" />
 	</joint>
 	<link name="${prefix}_appendix_link">

File: urdf/base_clause/base_clause.urdf.xacro (robot description, xacro)
@@ -12,4 +12,5 @@
 	  <limit lower="${-M_PI}" upper="${M_PI}" effort="${torque}" velocity="${velocity}" />
 	  <insert_block name="joint_axis"/>
+	  <dynamics friction="1.0" />
 	</joint>
 	<link name="${prefix}_base_clause_link">

File: urdf/coxa/coxa.urdf.xacro (robot description, xacro)
@@ -12,4 +12,5 @@
       <limit lower="-0.0" upper="0.0" effort="100" velocity="100" />
 	  <insert_block name="joint_axis"/>
+	  <dynamics friction="1.0" />
 	</joint>
 	<link name="${prefix}_coxa_link">

File: urdf/params/robot.xacro (robot description, xacro)
@@ -20,15 +20,15 @@
   <property name="RH_thigh_length" value="${thigh_length}"/>
   <property name="RH_tibia_length" value="${tibia_length}"/>
-  <property name="base_clause_radius" value="0.04"/>
-  <property name="thigh_radius" value="0.04"/>
-  <property name="tibia_radius" value="0.04"/>
-  <property name="appendix_radius" value="0.04"/>
+  <property name="base_clause_radius" value="0.05"/>
+  <property name="thigh_radius" value="0.05"/>
+  <property name="tibia_radius" value="0.05"/>
+  <property name="appendix_radius" value="0.05"/>
   <property name="base_clause_rho" value="${1240*0.1}"/>
   <property name="thigh_rho" value="${1240*0.1}"/>
   <property name="tibia_rho" value="${1240*0.1}"/>
   <property name="appendix_rho" value="${1240*0.1}"/>
-  <property name="base_clause_torque" value="50"/>
-  <property name="thigh_torque" value="50"/>
-  <property name="tibia_torque" value="50"/>
+  <property name="base_clause_torque" value="100"/>
+  <property name="thigh_torque" value="100"/>
+  <property name="tibia_torque" value="100"/>
   <property name="base_clause_velocity" value="100"/>
   <property name="thigh_velocity" value="100"/>

File: urdf/thigh/thigh.urdf.xacro (robot description, xacro)
@@ -12,4 +12,5 @@
 	  <limit lower="${-M_PI}" upper="${M_PI}" effort="${torque}" velocity="${velocity}" />
 	  <insert_block name="joint_axis"/>
+	  <dynamics friction="1.0" />
 	</joint>
 	<link name="${prefix}_thigh_link">
